File: ATmega64M1_Dev_Board.brd (EAGLE design)
At the start: 99.1 x 53.3 mm, 67 parts, among them IC1 LM1117IMPX-3.3, IC11 ATMEGA64M1TQFP32, IC2 LM1117IMPX-5.0, IC3 ADM3053M, IC4 FT232RL, J1 DCJ0202, Q1 16M, U1 MCP2562

Commit message: Minor fixes.
Routing:
- net XTAL2: track 12.2 -> 12.8 mm
Changed lines of the file:
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@@
 </element>
 <element name="IC11" library="ATmega64M1" package="QFP-32" value="ATMEGA64M1TQFP32" x="50.8" y="29.21" smashed="yes" rot="R180">
-<attribute name="NAME" x="48.57" y="32.584" size="1.27" layer="25"/>
-<attribute name="VALUE" x="48.07" y="32.115" size="0.4318" layer="27" rot="R180"/>
+<attribute name="NAME" x="54.483" y="24.765" size="1.27" layer="25" ratio="10" align="top-left"/>
+<attribute name="VALUE" x="53.594" y="36.576" size="1.27" layer="27" ratio="10" rot="R180"/>
 </element>
 <element name="X2" library="con-usb-3" package="USB-B-H" value="" x="6.35" y="38.1" smashed="yes"/>
@@
 </element>
 <element name="C9" library="rcl" library_urn="urn:adsk.eagle:library:334" package="C0603" package3d_urn="urn:adsk.eagle:package:23616/2" value="22p" x="35.56" y="32.385" smashed="yes" rot="R270">
-<attribute name="NAME" x="36.83" y="32.385" size="1.27" layer="25" rot="R270" align="bottom-center"/>
+<attribute name="NAME" x="36.83" y="30.48" size="1.27" layer="25" rot="R180"/>
 <attribute name="SPICEPREFIX" value="C" x="35.56" y="32.385" size="1.778" layer="27" rot="R270" display="off"/>
 <attribute name="VALUE" x="33.655" y="33.02" size="1.27" layer="27" rot="R270"/>
 </element>
 <element name="C11" library="rcl" library_urn="urn:adsk.eagle:library:334" package="C0603" package3d_urn="urn:adsk.eagle:package:23616/2" value="22p" x="35.56" y="26.67" smashed="yes" rot="R90">
-<attribute name="NAME" x="36.83" y="26.67" size="1.27" layer="25" rot="R270" align="bottom-center"/>
+<attribute name="NAME" x="37.465" y="24.765" size="1.27" layer="25" rot="R180"/>
 <attribute name="SPICEPREFIX" value="C" x="35.56" y="26.67" size="1.778" layer="27" rot="R90" display="off"/>
 <attribute name="VALUE" x="37.465" y="26.035" size="1.27" layer="27" rot="R90"/>
@@
 </element>
 <element name="R3" library="rcl" library_urn="urn:adsk.eagle:library:334" package="M0805" package3d_urn="urn:adsk.eagle:package:23556/1" value="10k" x="41.91" y="16.51" smashed="yes" rot="R90">
-<attribute name="NAME" x="41.275" y="20.32" size="1.27" layer="25"/>
+<attribute name="NAME" x="41.275" y="18.415" size="1.27" layer="25"/>
 <attribute name="SPICEPREFIX" value="R" x="41.91" y="16.51" size="1.778" layer="27" rot="R90" display="off"/>
 <attribute name="VALUE" x="44.45" y="15.24" size="1.27" layer="27" rot="R90"/>
@@
 <wire x1="18.03" y1="33.905" x2="18.415" y2="34.29" width="0.3048" layer="1"/>
 <via x="39.37" y="21.59" extent="1-16" drill="0.35"/>
-<via x="21.59" y="33.02" extent="1-16" drill="0.35"/>
+<via x="27.94" y="25.4" extent="1-16" drill="0.35"/>
 <via x="74.93" y="45.72" extent="1-16" drill="0.35"/>
 <via x="74.93" y="39.37" extent="1-16" drill="0.35"/>
@@
 <via x="52.705" y="29.845" extent="1-16" drill="0.35"/>
 <via x="48.26" y="30.48" extent="1-16" drill="0.35"/>
-<via x="36.83" y="24.13" extent="1-16" drill="0.35"/>
+<via x="33.02" y="30.48" extent="1-16" drill="0.35"/>
 <wire x1="50" y1="23.76" x2="50" y2="28.41" width="0.3048" layer="1"/>
 <wire x1="50" y1="28.41" x2="50.165" y2="28.575" width="0.3048" layer="1"/>
@@
 <wire x1="23.945" y1="32.605" x2="25.815" y2="32.605" width="0.3048" layer="1"/>
 <wire x1="25.815" y1="32.605" x2="26.67" y2="31.75" width="0.3048" layer="1"/>
-<wire x1="45.35" y1="29.21" x2="41.91" y2="29.21" width="0.3048" layer="1"/>
-<via x="41.91" y="29.21" extent="1-16" drill="0.35"/>
+<wire x1="45.35" y1="29.21" x2="41.275" y2="29.21" width="0.3048" layer="1"/>
+<via x="41.275" y="29.21" extent="1-16" drill="0.35"/>
 <wire x1="39.37" y1="36.83" x2="38.1" y2="36.83" width="0.3048" layer="16"/>
-<wire x1="41.91" y1="29.21" x2="41.91" y2="34.29" width="0.3048" layer="16"/>
-<wire x1="41.91" y1="34.29" x2="39.37" y2="36.83" width="0.3048" layer="16"/>
+<wire x1="41.275" y1="29.21" x2="41.275" y2="34.925" width="0.3048" layer="16"/>
+<wire x1="41.275" y1="34.925" x2="39.37" y2="36.83" width="0.3048" layer="16"/>
 <wire x1="38.1" y1="36.83" x2="31.75" y2="36.83" width="0.3048" layer="16"/>
 <wire x1="31.75" y1="36.83" x2="26.67" y2="31.75" width="0.3048" layer="16"/>
@@
 <wire x1="39.37" y1="26.797" x2="36.283" y2="26.797" width="0.3048" layer="1"/>
 <wire x1="36.283" y1="26.797" x2="35.56" y2="27.52" width="0.3048" layer="1"/>
-<wire x1="45.35" y1="30.01" x2="41.44" y2="30.01" width="0.3048" layer="1"/>
-<wire x1="41.44" y1="30.01" x2="40.64" y2="29.21" width="0.3048" layer="1"/>
-<wire x1="40.64" y1="29.21" x2="40.64" y2="27.94" width="0.3048" layer="1"/>
-<wire x1="40.64" y1="27.94" x2="40.513" y2="27.94" width="0.3048" layer="1"/>
-<wire x1="40.513" y1="27.94" x2="39.37" y2="26.797" width="0.3048" layer="1"/>
+<wire x1="45.35" y1="30.01" x2="40.17" y2="30.01" width="0.3048" layer="1"/>
+<wire x1="40.17" y1="30.01" x2="39.37" y2="29.21" width="0.3048" layer="1"/>
+<wire x1="39.37" y1="29.21" x2="39.37" y2="26.797" width="0.3048" layer="1"/>
 </signal>
 <signal name="AREF">
@@
 <wire x1="25.4" y1="14.175" x2="25.4" y2="17.78" width="0.508" layer="1"/>
 <wire x1="25.4" y1="17.78" x2="22.86" y2="20.32" width="0.508" layer="1"/>
-<wire x1="35.56" y1="12.7" x2="34.29" y2="13.97" width="0.4064" layer="1"/>
+<wire x1="35.56" y1="12.7" x2="33.579" y2="14.681" width="0.4064" layer="1"/>
 <wire x1="35.56" y1="2.54" x2="35.56" y2="12.7" width="0.4064" layer="1"/>
-<wire x1="34.29" y1="13.97" x2="31.75" y2="13.97" width="0.4064" layer="1"/>
-<wire x1="31.75" y1="13.97" x2="31.039" y2="14.681" width="0.4064" layer="1"/>
-<wire x1="31.039" y1="14.681" x2="30.48" y2="14.681" width="0.4064" layer="1"/>
+<wire x1="33.579" y1="14.681" x2="30.48" y2="14.681" width="0.4064" layer="1"/>
 <polygon width="0.3048" layer="1" isolate="0.4064">
 <vertex x="27.94" y="16.51"/>
