File: ATmega64M1_Dev_Board.sch (EAGLE design)
At the start: 67 parts, among them IC1 LM1117IMPX-3.3, IC11 ATMEGA64M1TQFP32, IC2 LM1117IMPX-5.0, IC3 ADM3053M, IC4 FT232RL, J1 DCJ0202, Q1 16M, U1 MCP2562

Commit message: Fixed ICSP pin allocation.
Connections:
- net A8: no longer SV1.4
- net D0_RX: now also SV1.3
- net D14: now also SV1.1
- net D1_TX: now also SV1.4
- net D5: no longer SV1.6
- net D6: no longer SV1.3
- net GND: now also SV1.6; no longer SV1.1
- net RST: now also SV1.5; no longer SV1.2
- net VCC: now also SV1.2; no longer SV1.5
Other:
- moved on the sheet: SV1
